File: Hardware/uartConverter.brd (EAGLE design)
At the start: 11 parts

Commit message: routage
Parts:
- added J8: (no value), con-amp:10X03MTA
- U$2: device STM32F4-DISCOVERY:STM32F4-DISCOVERY -> STM32F4-DISCOVERY_CF_INTECH:STM32F4-DISCOVERY
- moved X1 246.0 mm to (7.62, 77.5)
- moved J7 204.8 mm to (66.0, 80.0), turned to 90 degrees
- moved U$3 194.5 mm to (16.5, 22.9), turned to 90 degrees
- moved J6 190.4 mm to (53.3, 80.0), turned to 90 degrees
- moved J5 176.9 mm to (41.9, 80.0), turned to 90 degrees
- moved J4 164.4 mm to (31.8, 80.0), turned to 90 degrees
- moved J3 150.3 mm to (64.8, 3.81), turned to 270 degrees
- moved U$2 133.6 mm to (76.2, 41.9), turned to 270 degrees
- moved J2 126.3 mm to (41.9, 3.81), turned to 270 degrees
- moved J1 114.8 mm to (31.8, 3.81), turned to 270 degrees
- moved U$1 65.2 mm to (8.89, 43.2)
Connections:
- net 3.3V: now also U$2.VDD; no longer U$2.P$3
- net 5V: now also U$2.5V; no longer U$2.P$53
- net AX12_RX_TX: now also J8.3
- net ESP_RX: now also U$2.PC6
- net ESP_TX: now also U$2.PC7
- net GND: now also J8.1, U$2.GND, U$2.GND6; no longer U$2.P$1, U$2.P$51
- net STM_RX_TX: now also U$2.PA2, U$2.PA3; no longer U$2.P$13, U$2.P$14
- net VCC: now also J8.2
Routing:
- net AX12_RX_TX: track 0.00 -> 257.2 mm, vias 0 -> 2
- net VCC: track 0.00 -> 225.0 mm
- net 3.3V: track 0.00 -> 133.2 mm
- net 5V: track 0.00 -> 99.2 mm
- net STM_RX_TX: track 0.00 -> 77.8 mm
- net ESP_RX: track 0.00 -> 32.1 mm, vias 0 -> 2
- net ESP_TX: track 0.00 -> 15.3 mm
- added copper zone on layer 16, net GND
Other:
- board outline added: 100 x 88.9 mm
