File: Hardware/uartConverter.sch (EAGLE design)
At the start: 11 parts

Commit message: routage
Parts:
- added J8: (no value), con-amp:MTA03-100
- U$2: device STM32F4-DISCOVERY:STM32F4-DISCOVERY -> STM32F4-DISCOVERY_CF_INTECH:STM32F4-DISCOVERY
Connections:
- net AX12_RX_TX: now also J8.3
- net ESP_RX: now also U$2.PC6
- net ESP_TX: now also U$2.PC7
- net GND: now also J8.1
- net VCC: now also J8.2
Changed lines of the file:
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@@
 <parts>
 <part name="U$1" library="SparkFun-Boards" deviceset="LOGIC_LEVEL_CONVERTER" device=""/>
-<part name="U$2" library="STM32F4-DISCOVERY" deviceset="STM32F4-DISCOVERY" device=""/>
+<part name="U$2" library="STM32F4-DISCOVERY_CF_INTECH" deviceset="STM32F4-DISCOVERY" device=""/>
 <part name="J1" library="con-amp" deviceset="MTA03-100" device=""/>
 <part name="J2" library="con-amp" deviceset="MTA03-100" device=""/>
@@
 <part name="P+1" library="supply1" deviceset="VCC" device=""/>
 <part name="P+2" library="supply1" deviceset="VCC" device=""/>
+<part name="J8" library="con-amp" deviceset="MTA03-100" device=""/>
 </parts>
 <sheets>
@@
 <instance part="J6" gate="G$1" x="35.56" y="-66.04"/>
 <instance part="J7" gate="G$1" x="35.56" y="-73.66"/>
-<instance part="U$3" gate="G$1" x="-45.72" y="-60.96"/>
+<instance part="U$3" gate="G$1" x="-45.72" y="-60.96" smashed="yes">
+<attribute name="NAME" x="-58.42" y="-50.8" size="1.778" layer="95"/>
+<attribute name="VALUE" x="-58.42" y="-66.04" size="1.778" layer="95"/>
+</instance>
 <instance part="X1" gate="-1" x="22.86" y="-119.38" rot="R180"/>
 <instance part="X1" gate="-2" x="22.86" y="-114.3" rot="R180"/>
@@
 <instance part="P+1" gate="VCC" x="10.16" y="-109.22"/>
 <instance part="P+2" gate="VCC" x="30.48" y="-91.44"/>
+<instance part="J8" gate="G$1" x="35.56" y="-78.74"/>
 </instances>
 <busses>
@@
 <pinref part="J7" gate="G$1" pin="1"/>
 <wire x1="33.02" y1="-76.2" x2="33.02" y2="-68.58" width="0.1524" layer="91"/>
-<wire x1="33.02" y1="-83.82" x2="33.02" y2="-76.2" width="0.1524" layer="91"/>
+<wire x1="33.02" y1="-83.82" x2="33.02" y2="-81.28" width="0.1524" layer="91"/>
+<wire x1="33.02" y1="-81.28" x2="33.02" y2="-76.2" width="0.1524" layer="91"/>
 <wire x1="33.02" y1="-83.82" x2="20.32" y2="-83.82" width="0.1524" layer="91"/>
 <pinref part="SUPPLY2" gate="GND" pin="GND"/>
+<pinref part="J8" gate="G$1" pin="1"/>
+<junction x="33.02" y="-81.28"/>
 </segment>
 <segment>
@@
 <segment>
 <pinref part="J7" gate="G$1" pin="3"/>
-<wire x1="38.1" y1="-83.82" x2="38.1" y2="-76.2" width="0.1524" layer="91"/>
+<wire x1="38.1" y1="-83.82" x2="38.1" y2="-81.28" width="0.1524" layer="91"/>
 <pinref part="J6" gate="G$1" pin="3"/>
+<wire x1="38.1" y1="-81.28" x2="38.1" y2="-76.2" width="0.1524" layer="91"/>
 <wire x1="38.1" y1="-76.2" x2="38.1" y2="-68.58" width="0.1524" layer="91"/>
 <pinref part="J5" gate="G$1" pin="3"/>
@@
 <wire x1="38.1" y1="-83.82" x2="50.8" y2="-83.82" width="0.1524" layer="91"/>
 <label x="50.8" y="-83.82" size="1.778" layer="95"/>
+<pinref part="J8" gate="G$1" pin="3"/>
+<junction x="38.1" y="-81.28"/>
 </segment>
 <segment>
@@
 <label x="-76.2" y="-60.96" size="1.778" layer="95"/>
 </segment>
+<segment>
+<pinref part="U$2" gate="G$1" pin="PC6"/>
+<wire x1="17.78" y1="0" x2="10.16" y2="0" width="0.1524" layer="91"/>
+<label x="10.16" y="0" size="1.778" layer="95"/>
+</segment>
 </net>
 <net name="N$3" class="0">
@@
 <wire x1="-30.48" y1="-53.34" x2="-17.78" y2="-53.34" width="0.1524" layer="91"/>
 <label x="-17.78" y="-53.34" size="1.778" layer="95"/>
+</segment>
+<segment>
+<pinref part="U$2" gate="G$1" pin="PC7"/>
+<wire x1="48.26" y1="0" x2="55.88" y2="0" width="0.1524" layer="91"/>
+<label x="55.88" y="0" size="1.778" layer="95"/>
 </segment>
 </net>
@@
 <wire x1="30.48" y1="-93.98" x2="30.48" y2="-96.52" width="0.1524" layer="91"/>
 <pinref part="J7" gate="G$1" pin="2"/>
-<wire x1="35.56" y1="-96.52" x2="35.56" y2="-76.2" width="0.1524" layer="91"/>
+<wire x1="35.56" y1="-96.52" x2="35.56" y2="-81.28" width="0.1524" layer="91"/>
 <pinref part="J6" gate="G$1" pin="2"/>
+<wire x1="35.56" y1="-81.28" x2="35.56" y2="-76.2" width="0.1524" layer="91"/>
 <wire x1="35.56" y1="-76.2" x2="35.56" y2="-68.58" width="0.1524" layer="91"/>
 <pinref part="J5" gate="G$1" pin="2"/>
@@
 <wire x1="30.48" y1="-96.52" x2="35.56" y2="-96.52" width="0.1524" layer="91"/>
 <pinref part="P+2" gate="VCC" pin="VCC"/>
-</segment>
-</net>
+<pinref part="J8" gate="G$1" pin="2"/>
+<junction x="35.56" y="-81.28"/>
+</segment>
+</net>
